File: led-plate-96-well.kicad_pcb (KiCad board)
At the start: 2 copper layers, 166.3 x 99.1 mm, 127 parts, among them J2 RAPC722X, U1 R-78E5.0-0.5, U2 A000053, U3 WST2N7002, U4 WST2N7002, U5 WST2N7002, U6 WST2N7002

Commit message: set components and build again
Parts:
- R14, R20, R4, R8: value 100mΩ -> 100Ω
