File: basic-test/basic-test.kicad_sch (KiCad schematic)
At the start: 0 parts

Commit message: create basic test pcb
Parts:
- added D1, D10, D11, D12, D13, D14, D15, D16, D17, D18, D19, D2, D20, D21, D22, D23, D24, D25, D26, D27, D28, D29, D3, D30, D4, D5, D6, D7, D8, D9: Red, PCM_JLCPCB:D_0805, symbol PCM_JLCPCB-Diodes:LED,0805,Red
- added J1: RAPC722X, RAPC722X:SWITCHCRAFT_RAPC722X, symbol RAPC722X:RAPC722X
- added Q1: AO3400A, PCM_JLCPCB:Q_SOT-23, symbol PCM_JLCPCB-Transistors:NMOS,AO3400A
- added R1, R10, R11, R2, R3, R4, R5, R6, R7, R8, R9: 100Ω, PCM_JLCPCB:R_0603, symbol PCM_JLCPCB-Resistors:0603,100Ω
- added R12: 10kΩ, PCM_JLCPCB:R_0603, symbol PCM_JLCPCB-Resistors:0603,10kΩ
- added U1: A000053, A000053:A000053, symbol A000053:A000053
Connections:
- new net: D5.1, D6.2
- new net: Q1.1 (G), R11.1
- new net: Q1.3 (D), R1.1, R10.1, R2.1, R3.1, R4.1, R5.1, R6.1, R7.1, R8.1, R9.1
- new net: D23.1, D24.2
- new net: D4.1, D5.2
- new net: D29.1, D30.2
- new net: D28.1, D29.2
- new net: D8.1, D9.2
- new net: D7.1, D8.2
- new net: D13.2, R5.2
- new net: D22.1, D23.2
- new net: D22.2, R8.2
- new net: D10.2, R4.2
- new net: D20.1, D21.2
- new net: D17.1, D18.2
- new net: D16.1, D17.2
- new net: D11.1, D12.2
- new net: D14.1, D15.2
- new net: D13.1, D14.2
- new net: D16.2, R6.2
- new net: D19.2, R7.2
- new net: R11.2, R12.1, U1.10 (5(PWM))
- new net: D19.1, D20.2
- new net: D10.1, D11.2
- new net: D2.1, D3.2
- new net: D1.1, D2.2
- new net: D7.2, R3.2
- new net: D28.2, R10.2
- new net: D1.2, R1.2
- new net: D26.1, D27.2
- new net: D25.1, D26.2
- new net: D4.2, R2.2
- new net: D25.2, R9.2
- new net: U1.30 (RESET), U1.5 (RESET)
- new net +7.5V: J1.PIN, U1.32 (VIN)
- new net GND: D12.1, D15.1, D18.1, D21.1, D24.1, D27.1, D3.1, D30.1, D6.1, D9.1, J1.SLEEVE, Q1.2 (S), R12.2, U1.31 (GND), U1.6 (GND)
- no-connect marks 0 -> 28

Commit message: fix ciruit
Connections:
- net +7.5V: now also R1.1, R10.1, R2.1, R3.1, R4.1, R5.1, R6.1, R7.1, R8.1, R9.1
- net GND: no longer D12.1, D15.1, D18.1, D21.1, D24.1, D27.1, D3.1, D30.1, D6.1, D9.1
- new net: D12.1, D15.1, D18.1, D21.1, D24.1, D27.1, D3.1, D30.1, D6.1, D9.1, Q1.3 (D)
Changed lines of the file:
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@@
+	)
+	(junction
+		(at 167.64 54.61)
+		(diameter 0)
+		(color 0 0 0 0)
+	)
+	(junction
+		(at 246.38 35.56)
+		(diameter 0)
+		(color 0 0 0 0)
+	)
+	(junction
+		(at 66.04 124.46)
+		(diameter 0)
+		(color 0 0 0 0)
+	)
+	(junction
+		(at 78.74 124.46)
+		(diameter 0)
+		(color 0 0 0 0)
+	)
+	(junction
+		(at 104.14 54.61)
+		(diameter 0)
+		(color 0 0 0 0)
+	)
+	(junction
+		(at 91.44 54.61)
+		(diameter 0)
+		(color 0 0 0 0)
+	)
+	(junction
+		(at 255.27 35.56)
+		(diameter 0)
+		(color 0 0 0 0)
+	)
+	(junction
+		(at 256.54 35.56)
+		(diameter 0)
+		(color 0 0 0 0)
+	)
+	(junction
+		(at 142.24 124.46)
+		(diameter 0)
+		(color 0 0 0 0)
+	)
+	(junction
+		(at 252.73 48.26)
+		(diameter 0)
+		(color 0 0 0 0)
+	)
+	(junction
+		(at 154.94 54.61)
+		(diameter 0)
+		(color 0 0 0 0)
+	)
+	(junction
+		(at 104.14 124.46)
+		(diameter 0)
+		(color 0 0 0 0)
 	)
 	(junction
@@
 	)
 	(junction
-		(at 167.64 54.61)
-		(diameter 0)
-		(color 0 0 0 0)
-	)
-	(junction
-		(at 246.38 35.56)
-		(diameter 0)
-		(color 0 0 0 0)
-	)
-	(junction
-		(at 66.04 124.46)
-		(diameter 0)
-		(color 0 0 0 0)
-	)
-	(junction
-		(at 78.74 124.46)
-		(diameter 0)
-		(color 0 0 0 0)
-	)
-	(junction
-		(at 104.14 54.61)
-		(diameter 0)
-		(color 0 0 0 0)
-	)
-	(junction
-		(at 186.69 124.46)
-		(diameter 0)
-		(color 0 0 0 0)
-	)
-	(junction
-		(at 91.44 54.61)
-		(diameter 0)
-		(color 0 0 0 0)
-	)
-	(junction
-		(at 255.27 35.56)
-		(diameter 0)
-		(color 0 0 0 0)
-	)
-	(junction
-		(at 142.24 124.46)
-		(diameter 0)
-		(color 0 0 0 0)
-	)
-	(junction
-		(at 252.73 48.26)
-		(diameter 0)
-		(color 0 0 0 0)
-	)
-	(junction
-		(at 154.94 54.61)
-		(diameter 0)
-		(color 0 0 0 0)
-	)
-	(junction
-		(at 104.14 124.46)
-		(diameter 0)
-		(color 0 0 0 0)
-	)
-	(junction
 		(at 246.38 40.64)
 		(diameter 0)
@@
 	(wire
 		(pts
-			(xy 167.64 124.46) (xy 186.69 124.46)
-		)
-		(stroke
-			(width 0)
-			(type default)
-		)
-	)
-	(wire
-		(pts
 			(xy 53.34 54.61) (xy 53.34 76.2)
 		)
@@
 	(wire
 		(pts
+			(xy 256.54 35.56) (xy 261.62 35.56)
+		)
+		(stroke
+			(width 0)
+			(type default)
+		)
+	)
+	(wire
+		(pts
+			(xy 167.64 124.46) (xy 177.8 124.46)
+		)
+		(stroke
+			(width 0)
+			(type default)
+		)
+	)
+	(wire
+		(pts
 			(xy 66.04 54.61) (xy 53.34 54.61)
 		)
@@
 	(wire
 		(pts
+			(xy 261.62 26.67) (xy 167.64 26.67)
+		)
+		(stroke
+			(width 0)
+			(type default)
+		)
+	)
+	(wire
+		(pts
 			(xy 154.94 106.68) (xy 154.94 124.46)
 		)
@@
 	(wire
 		(pts
+			(xy 177.8 54.61) (xy 181.61 54.61)
+		)
+		(stroke
+			(width 0)
+			(type default)
+		)
+	)
+	(wire
+		(pts
+			(xy 177.8 124.46) (xy 177.8 54.61)
+		)
+		(stroke
+			(width 0)
+			(type default)
+		)
+	)
+	(wire
+		(pts
 			(xy 91.44 124.46) (xy 104.14 124.46)
 		)
@@
 	(wire
 		(pts
+			(xy 261.62 35.56) (xy 261.62 26.67)
+		)
+		(stroke
+			(width 0)
+			(type default)
+		)
+	)
+	(wire
+		(pts
 			(xy 243.84 35.56) (xy 246.38 35.56)
 		)
@@
 	(wire
 		(pts
+			(xy 167.64 26.67) (xy 167.64 54.61)
+		)
+		(stroke
+			(width 0)
+			(type default)
+		)
+	)
+	(wire
+		(pts
 			(xy 154.94 54.61) (xy 142.24 54.61)
 		)
@@
 		)
 		(stroke
-			(width 0)
-			(type default)
-		)
-	)
-	(wire
-		(pts
-			(xy 181.61 54.61) (xy 167.64 54.61)
-		)
-		(stroke
