File: led-plate-96-well/led-plate-96-well.kicad_sch (KiCad schematic)
At the start: 2 parts, among them U1 TLC5947RHB, U2 A000053

Commit message: start main board
Parts:
- added C1: 100nF, Capacitor_SMD:C_0603_1608Metric, symbol Device:C
- added C2: 10uF, Capacitor_SMD:C_0805_2012Metric, symbol Device:C
- added D1, D10, D11, D12, D13, D14, D15, D16, D17, D18, D19, D2, D20, D21, D22, D23, D24, D3, D4, D5, D6, D7, D8, D9: LED, SMD2835_WITH_STEP:LED_PLCC_2835, symbol Device:LED
- added J1: RAPC722X, RAPC722X:SWITCHCRAFT_RAPC722X, symbol RAPC722X:RAPC722X
- added R1: 2.49kΩ, Resistor_SMD:R_0402_1005Metric, symbol Device:R
- added R2: 10kΩ, Resistor_SMD:R_0603_1608Metric, symbol Device:R
- renumbered U2 to U1, U1 to U2
Connections:
- net at U1.10 (5(PWM)): now also U2.31 (SCLK)
- net at U1.11 (6(PWM)/A7): now also U2.30 (BLANK), R2.2
- net at U1.14 (9(PWM)/A9): now also U2.26 (XLAT)
- net +5V: now reaches U1.29 (+5V)
- net +5V: now also U2.28 (VCC), C1.2, C2.2, D1.2 (A), D10.2 (A), D11.2 (A), D12.2 (A), D13.2 (A), D14.2 (A), D15.2 (A), D16.2 (A), D17.2 (A), D18.2 (A), D19.2 (A), D2.2 (A), D20.2 (A), D21.2 (A), D22.2 (A), D23.2 (A), D24.2 (A), D3.2 (A), D4.2 (A), D5.2 (A), D6.2 (A), D7.2 (A), D8.2 (A), D9.2 (A), J1.PIN, R2.1
- net GND: now reaches U1.31 (GND), U1.6 (GND)
- net GND: now also U2.29 (GND), U2.33 (PowerPAD), C1.1, C2.1, J1.SLEEVE, R1.1
- net at U1.8 (3(PWM)/SCL): now also U2.32 (SIN)
- net at U2.1 (OUT0): now also D1.1 (K)
- net at U2.10 (OUT9): now also D10.1 (K)
- net at U2.11 (OUT10): now also D11.1 (K)
- net at U2.12 (OUT11): now also D12.1 (K)
- net at U2.13 (OUT12): now also D13.1 (K)
- net at U2.14 (OUT13): now also D14.1 (K)
- net at U2.15 (OUT14): now also D15.1 (K)
- net at U2.16 (OUT15): now also D16.1 (K)
- net at U2.17 (OUT16): now also D17.1 (K)
- net at U2.18 (OUT17): now also D18.1 (K)
- net at U2.19 (OUT18): now also D19.1 (K)
- net at U2.2 (OUT1): now also D2.1 (K)
- net at U2.20 (OUT19): now also D20.1 (K)
- net at U2.21 (OUT20): now also D21.1 (K)
- net at U2.22 (OUT21): now also D22.1 (K)
- net at U2.23 (OUT22): now also D23.1 (K)
- net at U2.24 (OUT23): now also D24.1 (K)
- net at U2.27 (IREF): now also R1.2
- net at U2.3 (OUT2): now also D3.1 (K)
- net at U2.4 (OUT3): now also D4.1 (K)
- net at U2.5 (OUT4): now also D5.1 (K)
- net at U2.6 (OUT5): now also D6.1 (K)
- net at U2.7 (OUT6): now also D7.1 (K)
- net at U2.8 (OUT7): now also D8.1 (K)
- net at U2.9 (OUT8): now also D9.1 (K)
Other:
- moved on the sheet: U1, U2

Commit message: layout leds
Parts:
- added C10, C11, C13, C4, C5, C7, C8: 10uF, Capacitor_SMD:C_0805_2012Metric, symbol Device:C
- added C12, C6, C9: 100nF, Capacitor_SMD:C_0603_1608Metric, symbol Device:C
- added C3: 100uF, Capacitor_SMD:C_1206_3216Metric, symbol Device:C
- added D25, D26, D27, D28, D29, D30, D31, D32, D33, D34, D35, D36, D37, D38, D39, D40, D41, D42, D43, D44, D45, D46, D47, D48, D49, D50, D51, D52, D53, D54, D55, D56, D57, D58, D59, D60, D61, D62, D63, D64, D65, D66, D67, D68, D69, D70, D71, D72, D73, D74, D75, D76, D77, D78, D79, D80, D81, D82, D83, D84, D85, D86, D87, D88, D89, D90, D91, D92, D93, D94, D95, D96: LED, SMD2835_WITH_STEP:LED_PLCC_2835, symbol Device:LED
- added R4, R6, R8: 2.49kΩ, Resistor_SMD:R_0402_1005Metric, symbol Device:R
- added U3, U4, U5: TLC5947RHB, Package_DFN_QFN:QFN-32-1EP_5x5mm_P0.5mm_EP3.45x3.45mm, symbol Driver_LED:TLC5947RHB
Connections:
- net +5V: now also C10.2, C11.2, C12.2, C13.2, C3.1, C4.2, C5.2, C6.2, C7.2, C8.2, C9.2, D25.2 (A), D26.2 (A), D27.2 (A), D28.2 (A), D29.2 (A), D30.2 (A), D31.2 (A), D32.2 (A), D33.2 (A), D34.2 (A), D35.2 (A), D36.2 (A), D37.2 (A), D38.2 (A), D39.2 (A), D40.2 (A), D41.2 (A), D42.2 (A), D43.2 (A), D44.2 (A), D45.2 (A), D46.2 (A), D47.2 (A), D48.2 (A), D49.2 (A), D50.2 (A), D51.2 (A), D52.2 (A), D53.2 (A), D54.2 (A), D55.2 (A), D56.2 (A), D57.2 (A), D58.2 (A), D59.2 (A), D60.2 (A), D61.2 (A), D62.2 (A), D63.2 (A), D64.2 (A), D65.2 (A), D66.2 (A), D67.2 (A), D68.2 (A), D69.2 (A), D70.2 (A), D71.2 (A), D72.2 (A), D73.2 (A), D74.2 (A), D75.2 (A), D76.2 (A), D77.2 (A), D78.2 (A), D79.2 (A), D80.2 (A), D81.2 (A), D82.2 (A), D83.2 (A), D84.2 (A), D85.2 (A), D86.2 (A), D87.2 (A), D88.2 (A), D89.2 (A), D90.2 (A), D91.2 (A), D92.2 (A), D93.2 (A), D94.2 (A), D95.2 (A), D96.2 (A), U3.28 (VCC), U4.28 (VCC), U5.28 (VCC)
- net GND: now also C10.1, C11.1, C12.1, C13.1, C3.2, C4.1, C5.1, C6.1, C7.1, C8.1, C9.1, R4.1, R6.1, R8.1, U3.29 (GND), U3.33 (PowerPAD), U4.29 (GND), U4.33 (PowerPAD), U5.29 (GND), U5.33 (PowerPAD)
- net at R2.2, U1.11 (6(PWM)/A7), U2.30 (BLANK): now also U3.30 (BLANK), U4.30 (BLANK), U5.30 (BLANK)
- net at U1.10 (5(PWM)), U2.31 (SCLK): now also U3.31 (SCLK), U4.31 (SCLK), U5.31 (SCLK)
- net at U1.14 (9(PWM)/A9), U2.26 (XLAT): now also U3.26 (XLAT), U4.26 (XLAT), U5.26 (XLAT)
- net at U2.25 (SOUT): now also U3.32 (SIN)
- new net: D75.1 (K), U5.3 (OUT2)
- new net: D37.1 (K), U3.13 (OUT12)
- new net: R8.2, U5.27 (IREF)
- new net: D60.1 (K), U4.12 (OUT11)
- new net: D54.1 (K), U4.6 (OUT5)
- new net: D84.1 (K), U5.12 (OUT11)
- new net: D46.1 (K), U3.22 (OUT21)
- new net: D93.1 (K), U5.21 (OUT20)
- new net: D40.1 (K), U3.16 (OUT15)
- new net: D69.1 (K), U4.21 (OUT20)
- new net: D80.1 (K), U5.8 (OUT7)
- new net: D66.1 (K), U4.18 (OUT17)
- new net: D89.1 (K), U5.17 (OUT16)
- new net: D83.1 (K), U5.11 (OUT10)
- new net: D31.1 (K), U3.7 (OUT6)
- new net: D67.1 (K), U4.19 (OUT18)
- new net: D87.1 (K), U5.15 (OUT14)
- new net: D43.1 (K), U3.19 (OUT18)
- new net: D82.1 (K), U5.10 (OUT9)
- new net: D76.1 (K), U5.4 (OUT3)
- new net: D81.1 (K), U5.9 (OUT8)
- new net: D44.1 (K), U3.20 (OUT19)
- new net: D35.1 (K), U3.11 (OUT10)
- new net: D53.1 (K), U4.5 (OUT4)
- new net: D61.1 (K), U4.13 (OUT12)
- new net: D96.1 (K), U5.24 (OUT23)
- new net: D85.1 (K), U5.13 (OUT12)
- new net: D70.1 (K), U4.22 (OUT21)
- new net: D88.1 (K), U5.16 (OUT15)
- new net: D57.1 (K), U4.9 (OUT8)
- new net: D49.1 (K), U4.1 (OUT0)
- new net: D48.1 (K), U3.24 (OUT23)
- new net: D34.1 (K), U3.10 (OUT9)
- new net: D73.1 (K), U5.1 (OUT0)
- new net: D86.1 (K), U5.14 (OUT13)
- new net: D90.1 (K), U5.18 (OUT17)
- new net: D91.1 (K), U5.19 (OUT18)
- new net: D74.1 (K), U5.2 (OUT1)
- new net: D92.1 (K), U5.20 (OUT19)
- new net: D94.1 (K), U5.22 (OUT21)
- new net: D95.1 (K), U5.23 (OUT22)
- new net: U4.25 (SOUT), U5.32 (SIN)
- new net: D77.1 (K), U5.5 (OUT4)
- new net: D78.1 (K), U5.6 (OUT5)
- new net: D79.1 (K), U5.7 (OUT6)
- new net: R4.2, U3.27 (IREF)
- new net: D58.1 (K), U4.10 (OUT9)
- new net: D59.1 (K), U4.11 (OUT10)
- new net: D62.1 (K), U4.14 (OUT13)
- new net: D63.1 (K), U4.15 (OUT14)
- new net: D64.1 (K), U4.16 (OUT15)
- new net: D65.1 (K), U4.17 (OUT16)
- new net: D50.1 (K), U4.2 (OUT1)
- new net: D68.1 (K), U4.20 (OUT19)
- new net: D71.1 (K), U4.23 (OUT22)
- new net: D72.1 (K), U4.24 (OUT23)
- new net: R6.2, U4.27 (IREF)
- new net: D51.1 (K), U4.3 (OUT2)
- new net: U3.25 (SOUT), U4.32 (SIN)
- new net: D52.1 (K), U4.4 (OUT3)
- new net: D55.1 (K), U4.7 (OUT6)
- new net: D56.1 (K), U4.8 (OUT7)
- new net: D32.1 (K), U3.8 (OUT7)
- new net: D36.1 (K), U3.12 (OUT11)
- new net: D29.1 (K), U3.5 (OUT4)
- new net: D47.1 (K), U3.23 (OUT22)
- new net: D27.1 (K), U3.3 (OUT2)
- new net: D26.1 (K), U3.2 (OUT1)
- new net: D30.1 (K), U3.6 (OUT5)
- new net: D25.1 (K), U3.1 (OUT0)
- new net: D42.1 (K), U3.18 (OUT17)
- new net: D41.1 (K), U3.17 (OUT16)
- new net: D33.1 (K), U3.9 (OUT8)
- new net: D38.1 (K), U3.14 (OUT13)
- new net: D28.1 (K), U3.4 (OUT3)
- new net: D39.1 (K), U3.15 (OUT14)
- new net: D45.1 (K), U3.21 (OUT20)
- no-connect marks 0 -> 26
Other:
- moved on the sheet: R2

Commit message: start redesign as 2 layer board
Parts:
- C3: value 100uF -> 10uF; footprint Capacitor_SMD:C_1206_3216Metric -> Capacitor_SMD:C_0805_2012Metric; part number CL31A107MQHNNNE -> CL21A106KAYNNNE
- R1: footprint Resistor_SMD:R_0402_1005Metric -> Resistor_SMD:R_0603_1608Metric; part number RTT022491FTH -> RC0603FR-072K49L
Changed lines of the file:
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@@
 			)
 		)
-		(property "Footprint" "Resistor_SMD:R_0402_1005Metric"
+		(property "Footprint" "Resistor_SMD:R_0603_1608Metric"
 			(at 210.82 112.268 90)
 			(effects
@@
 			)
 		)
-		(property "part number" "RTT022491FTH"
+		(property "part number" "RC0603FR-072K49L"
 			(at 210.82 110.49 0)
 			(effects
@@
 			)
 		)
-		(property "Value" "100uF"
+		(property "Value" "10uF"
 			(at 105.41 95.2499 0)
 			(effects
@@
 			)
 		)
-		(property "Footprint" "Capacitor_SMD:C_1206_3216Metric"
+		(property "Footprint" "Capacitor_SMD:C_0805_2012Metric"
 			(at 102.5652 97.79 0)
 			(effects
@@
 			)
 		)
-		(property "part number" "CL31A107MQHNNNE"
+		(property "part number" "CL21A106KAYNNNE"
 			(at 101.6 93.98 0)
 			(effects

Commit message: fix some part numbers and footprints
Parts:
- R4, R6, R8: footprint Resistor_SMD:R_0402_1005Metric -> Resistor_SMD:R_0603_1608Metric; part number RTT022491FTH -> RC0603FR-072K49L
Changed lines of the file:
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@@
 			)
 		)
-		(property "Footprint" "Resistor_SMD:R_0402_1005Metric"
+		(property "Footprint" "Resistor_SMD:R_0603_1608Metric"
 			(at 740.41 112.268 90)
 			(effects
@@
 			)
 		)
-		(property "part number" "RTT022491FTH"
+		(property "part number" "RC0603FR-072K49L"
 			(at 740.41 110.49 0)
 			(effects
@@
 			)
 		)
-		(property "Footprint" "Resistor_SMD:R_0402_1005Metric"
+		(property "Footprint" "Resistor_SMD:R_0603_1608Metric"
 			(at 384.81 109.728 90)
 			(effects
@@
 			)
 		)
-		(property "part number" "RTT022491FTH"
+		(property "part number" "RC0603FR-072K49L"
 			(at 384.81 107.95 0)
 			(effects
@@
 			)
 		)
-		(property "Footprint" "Resistor_SMD:R_0402_1005Metric"
+		(property "Footprint" "Resistor_SMD:R_0603_1608Metric"
 			(at 560.07 108.458 90)
 			(effects
@@
 			)
 		)
-		(property "part number" "RTT022491FTH"
+		(property "part number" "RC0603FR-072K49L"
 			(at 560.07 106.68 0)
 			(effects
